Commit message: Primer intento de camara

File: proyecto_final_rcsv/urdf/kobuki.urdf.xacro (robot description, xacro)
@@ -9,4 +9,5 @@
   <xacro:include filename="$(find proyecto_final_rcsv)/urdf/common_properties.urdf.xacro"/>
   <xacro:include filename="$(find proyecto_final_rcsv)/urdf/kobuki_gazebo.urdf.xacro"/>
+  <xacro:property name="camera_link" value="0.1" /> <!-- Size of square 'camera' box -->
   <!-- Kobuki -->
   <xacro:macro name="kobuki">
@@ -208,4 +209,75 @@
       </inertial>
     </link>
+    <!-- JUNTURA DE CAMARA -->
+    <joint name="camera_joint" type="fixed">
+      <axis xyz="0 1 0" />
+      <origin xyz="0 0 0.15" rpy="0 1.5708 0"/>
+      <parent link="base_link"/>
+      <child link="camera_link"/>
+    </joint>
+    <!-- Camera -->
+    <link name="camera_link">
+      <collision>
+        <origin xyz="0 0 0" rpy="0 0 0"/>
+        <geometry>
+          <box size="${camera_link} ${camera_link} ${camera_link}"/>
+        </geometry>
+      </collision>
+      <visual>
+        <origin xyz="0 0 0" rpy="0 0 0"/>
+        <geometry>
+          <box size="${camera_link} ${camera_link} ${camera_link}"/>
+        </geometry>
+        <material name="red">
+          <color rgba="1.0 0.0 0.0 1.0"/>
+        </material>
+      </visual>
+      <inertial>
+        <mass value="1e-5" />
+        <origin xyz="0 0 0" rpy="0 0 0"/>
+        <inertia ixx="1e-6" ixy="0" ixz="0" iyy="1e-6" iyz="0" izz="1e-6" />
+      </inertial>
+    </link>
+    <!-- Plugin de la camara -->
+    <gazebo reference="camera_link">
+    <sensor type="camera" name="camera_principal">
+      <update_rate>30.0</update_rate>
+      <visualize>true</visualize>
+      <camera name="head">
+        <horizontal_fov>1.3962634</horizontal_fov>
+        <image>
+          <width>800</width>
+          <height>800</height>
+          <format>R8G8B8</format>
+        </image>
+        <clip>
+          <near>0.02</near>
+          <far>300</far>
+        </clip>
+        <noise>
+          <type>gaussian</type>
+          <!-- Noise is sampled independently per pixel on each frame.
+               That pixel's noise value is added to each of its color
+               channels, which at that point lie in the range [0,1]. -->
+          <mean>0.0</mean>
+          <stddev>0.007</stddev>
+        </noise>
+      </camera>
+      <plugin name="camera_controller" filename="libgazebo_ros_camera.so">
+        <alwaysOn>true</alwaysOn>
+        <updateRate>0.0</updateRate>
+        <cameraName>kobuki/camera_principal</cameraName>
+        <imageTopicName>image_raw</imageTopicName>
+        <cameraInfoTopicName>camera_info</cameraInfoTopicName>
+        <frameName>camera_link</frameName>
+        <hackBaseline>0.07</hackBaseline>
+        <distortionK1>0.0</distortionK1>
+        <distortionK2>0.0</distortionK2>
+        <distortionK3>0.0</distortionK3>
+        <distortionT1>0.0</distortionT1>
+        <distortionT2>0.0</distortionT2>
+      </plugin>
+    </sensor>
+    </gazebo>
     <!-- Kobuki Gazebo simulation details -->
     <xacro:kobuki_sim/>

Commit message: Se finaliza la implementación de la camara de manera satisfactoria

File: proyecto_final_rcsv/urdf/kobuki.urdf.xacro (robot description, xacro)
@@ -212,5 +212,5 @@
     <joint name="camera_joint" type="fixed">
       <axis xyz="0 1 0" />
-      <origin xyz="0 0 0.15" rpy="0 1.5708 0"/>
+      <origin xyz="0.13 0 0.13" rpy="0 0 0"/>
       <parent link="base_link"/>
       <child link="camera_link"/>
@@ -241,42 +241,33 @@
     <!-- Plugin de la camara -->
     <gazebo reference="camera_link">
-    <sensor type="camera" name="camera_principal">
-      <update_rate>30.0</update_rate>
-      <visualize>true</visualize>
-      <camera name="head">
-        <horizontal_fov>1.3962634</horizontal_fov>
-        <image>
-          <width>800</width>
-          <height>800</height>
-          <format>R8G8B8</format>
-        </image>
-        <clip>
-          <near>0.02</near>
-          <far>300</far>
-        </clip>
-        <noise>
-          <type>gaussian</type>
-          <!-- Noise is sampled independently per pixel on each frame.
-               That pixel's noise value is added to each of its color
-               channels, which at that point lie in the range [0,1]. -->
-          <mean>0.0</mean>
-          <stddev>0.007</stddev>
-        </noise>
-      </camera>
-      <plugin name="camera_controller" filename="libgazebo_ros_camera.so">
-        <alwaysOn>true</alwaysOn>
-        <updateRate>0.0</updateRate>
-        <cameraName>kobuki/camera_principal</cameraName>
-        <imageTopicName>image_raw</imageTopicName>
-        <cameraInfoTopicName>camera_info</cameraInfoTopicName>
-        <frameName>camera_link</frameName>
-        <hackBaseline>0.07</hackBaseline>
-        <distortionK1>0.0</distortionK1>
-        <distortionK2>0.0</distortionK2>
-        <distortionK3>0.0</distortionK3>
-        <distortionT1>0.0</distortionT1>
-        <distortionT2>0.0</distortionT2>
-      </plugin>
-    </sensor>
+      <sensor type="camera" name="camara_principal">
+        <update_rate>30.0</update_rate>
+        <camera name="head">
+          <horizontal_fov>1.3962634</horizontal_fov>
+          <image>
+            <width>800</width>
+            <height>800</height>
+            <format>R8G8B8</format>
+          </image>
+          <clip>
+            <near>0.02</near>
+            <far>300</far>
+          </clip>
+        </camera>
+        <plugin name="camera_controller" filename="libgazebo_ros_camera.so">
+          <alwaysOn>true</alwaysOn>
+          <updateRate>0.0</updateRate>
+          <cameraName>kobuki/camara_principal</cameraName>
+          <imageTopicName>image_raw</imageTopicName>
+          <cameraInfoTopicName>camera_info</cameraInfoTopicName>
+          <frameName>camera_link</frameName>
+          <hackBaseline>0.07</hackBaseline>
+          <distortionK1>0.0</distortionK1>
+          <distortionK2>0.0</distortionK2>
+          <distortionK3>0.0</distortionK3>
+          <distortionT1>0.0</distortionT1>
+          <distortionT2>0.0</distortionT2>
+        </plugin>
+      </sensor>
     </gazebo>
     <!-- Kobuki Gazebo simulation details -->

Commit message: Se implementa la captura de imagenes de la camara en gazebo por medio de ros. ver test_camara.py

File: proyecto_final_rcsv/urdf/kobuki.urdf.xacro (robot description, xacro)
@@ -9,5 +9,5 @@
   <xacro:include filename="$(find proyecto_final_rcsv)/urdf/common_properties.urdf.xacro"/>
   <xacro:include filename="$(find proyecto_final_rcsv)/urdf/kobuki_gazebo.urdf.xacro"/>
-  <xacro:property name="camera_link" value="0.1" /> <!-- Size of square 'camera' box -->
+  <xacro:property name="camera_link" value="0.05" />
   <!-- Kobuki -->
   <xacro:macro name="kobuki">
@@ -212,5 +212,5 @@
     <joint name="camera_joint" type="fixed">
       <axis xyz="0 1 0" />
-      <origin xyz="0.13 0 0.13" rpy="0 0 0"/>
+      <origin xyz="0.13 0 0.115" rpy="0 0 0"/>
       <parent link="base_link"/>
       <child link="camera_link"/>
@@ -255,4 +255,5 @@
           </clip>
         </camera>
+          <visualize>true</visualize>
         <plugin name="camera_controller" filename="libgazebo_ros_camera.so">
           <alwaysOn>true</alwaysOn>
@@ -270,4 +271,5 @@
         </plugin>
       </sensor>
+      <material>Gazebo/RedTransparentOverlay</material>
     </gazebo>
     <!-- Kobuki Gazebo simulation details -->
